File: PCB/pepuino75.kicad_pcb (KiCad board)
At the start: 2 copper layers, 338.1 x 116.7 mm, 197 parts, among them SW1 Switch, SW10 Switch, SW11 Switch, SW12 Switch, SW13 Switch, SW14 Switch, SW15 Switch, SW16 Switch, SW17 Switch, SW18 Switch, SW19 Switch, SW2 Switch, SW20 Switch, SW21 Switch, SW22 Switch, SW23 Switch, SW24 Switch, SW25 Switch, SW26 Switch, SW27 Switch, SW28 Switch, SW29 Switch, SW3 Switch, SW30 Switch, SW31 Switch, SW32 Switch, SW33 Switch, SW34 Switch, SW35 Switch, SW36 Switch, SW37 Switch, SW38 Switch, SW39 Switch, SW4 Switch, SW40 Switch, SW41 Switch, SW42 Switch, SW43 Switch, SW44 Switch, SW45 Switch, SW46 Switch, SW47 Switch, SW48 Switch, SW49 Switch, SW5 Switch, SW50 Switch, SW51 Switch, SW52 Switch, SW53 Switch, SW54 Switch, SW55 Switch, SW56 Switch, SW57 Switch, SW58 Switch, SW59 Switch, SW6 Switch, SW60 Switch, SW61 Switch, SW62 Switch, SW63 Switch, SW64 Switch, SW65 Switch, SW66 Switch, SW67 Switch, SW68 Switch, SW69 Switch, SW7 Switch, SW71 Switch, SW72 Switch, SW73 Switch, SW74 Switch, SW75 Switch, SW76 Switch, SW77 Switch, SW78 Switch, SW79 Switch, SW8 Switch, SW80 Switch, SW81 Switch, SW82 Switch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

Commit message: update images and add silkscreen pcb
Parts:
- removed H1, H10, H11, H12, H13, H14, H15, H17, H18, H19, H2, H20, H22, H23, H24, H25, H3, H4, H5, H6, H7, H8, H9: MountingHole, MountingHole:MountingHole_2.2mm_M2
Routing:
- net ROW3: track 472.5 -> 426.9 mm, vias 12 -> 14
- net ROW4: track 424.1 -> 408.5 mm
- net ROW2: track 413.2 -> 401.6 mm
- net COL10: track 347.9 -> 353.3 mm
- net ROW0: track 392.4 -> 397.5 mm
- net COL13: track 388.3 -> 392.0 mm, vias 0 -> 2
- net COL9: track 333.0 -> 329.6 mm
- net rotaryA: track 305.8 -> 309.1 mm
- net COL6: track 284.8 -> 287.8 mm
- net COL0: track 137.2 -> 134.4 mm
- net COL8: track 285.8 -> 283.1 mm
- net COL1: track 178.7 -> 176.4 mm
- net COL5: track 247.0 -> 244.9 mm
- net COL7: track 272.4 -> 274.1 mm
- net ROW1: track 400.3 -> 398.9 mm
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Other:
- outline, holes or cut-outs redrawn
