File: PCB/PepuinoNova75.kicad_pcb (KiCad board)
At the start: 2 copper layers, 338.1 x 116.7 mm, 174 parts, among them SW1 Switch, SW10 Switch, SW11 Switch, SW12 Switch, SW13 Switch, SW14 Switch, SW15 Switch, SW16 Switch, SW17 Switch, SW18 Switch, SW19 Switch, SW2 Switch, SW20 Switch, SW21 Switch, SW22 Switch, SW23 Switch, SW24 Switch, SW25 Switch, SW26 Switch, SW27 Switch, SW28 Switch, SW29 Switch, SW3 Switch, SW30 Switch, SW31 Switch, SW32 Switch, SW33 Switch, SW34 Switch, SW35 Switch, SW36 Switch, SW37 Switch, SW38 Switch, SW39 Switch, SW4 Switch, SW40 Switch, SW41 Switch, SW42 Switch, SW43 Switch, SW44 Switch, SW45 Switch, SW46 Switch, SW47 Switch, SW48 Switch, SW49 Switch, SW5 Switch, SW50 Switch, SW51 Switch, SW52 Switch, SW53 Switch, SW54 Switch, SW55 Switch, SW56 Switch, SW57 Switch, SW58 Switch, SW59 Switch, SW6 Switch, SW60 Switch, SW61 Switch, SW62 Switch, SW63 Switch, SW64 Switch, SW65 Switch, SW66 Switch, SW67 Switch, SW68 Switch, SW69 Switch, SW7 Switch, SW71 Switch, SW72 Switch, SW73 Switch, SW74 Switch, SW75 Switch, SW76 Switch, SW77 Switch, SW78 Switch, SW79 Switch, SW8 Switch, SW80 Switch, SW81 Switch, SW82 Switch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

Commit message: fix fatal error in pcb +  fix case + update images
Parts:
- removed S5: MX_stab, ScottoKeebs_Stabilizers:Stabilizer_MX_2.00u
Connections:
- SW72 pad 1: unconnected-(SW72-Pad1) -> COL13
Routing:
- net COL12: track 399.9 -> 373.9 mm
Changed lines of the file:
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@@
 			(layers "*.Cu" "*.Mask")
 			(remove_unused_layers no)
-			(net "unconnected-(SW72-Pad1)")
+			(net "COL13")
 			(pinfunction "1_1")
 			(pintype "passive")
@@
 		)
 	)
-	(footprint "ScottoKeebs_Stabilizers:Stabilizer_MX_2.00u"
-		(layer "F.Cu")
-		(at 240.4745 -66.8338)
-		(descr "MX PCB Stabilizer 2.00u 2.25u 2.50u 2.75u")
-		(tags "MX Keyboard Stabilizer 2.00u 2.25u 2.50u 2.75u Cutout")
-		(property "Reference" "S5"
-			(at 0 -2 0)
-			(layer "F.SilkS")
-			(effects
-				(font
-					(size 1 1)
-					(thickness 0.15)
-				)
-			)
-		)
-		(property "Value" "MX_stab"
-			(at 0 2 0)
-			(layer "F.Fab")
-			(effects
-				(font
-					(size 1 1)
-					(thickness 0.15)
-				)
-			)
-		)
-		(property "Datasheet" ""
-			(at 0 0 0)
-			(layer "F.Fab")
-			(hide yes)
-			(effects
-				(font
-					(size 1.27 1.27)
-					(thickness 0.15)
-				)
-			)
-		)
-		(property "Description" "Cherry MX-style stabilizer"
-			(at 0 0 0)
-			(layer "F.Fab")
-			(hide yes)
-			(effects
-				(font
-					(size 1.27 1.27)
-					(thickness 0.15)
-				)
-			)
-		)
-		(sheetname "/")
-		(sheetfile "PepuinoNova75.kicad_sch")
-		(units
-			(unit
-				(name "A")
-				(pins)
-			)
-		)
-		(duplicate_pad_numbers_are_jumpers no)
-		(fp_line
-			(start -2 0)
-			(end 2 0)
-			(stroke
-				(width 0.1)
-				(type solid)
-			)
-			(layer "Dwgs.User")
-		)
-		(fp_line
-			(start 0 2)
-			(end 0 -2)
-			(stroke
-				(width 0.1)
-				(type solid)
-			)
-			(layer "Dwgs.User")
-		)
-		(fp_line
-			(start -15.313 -5.53)
-			(end -15.313 6.77)
-			(stroke
-				(width 0.1)
-				(type solid)
-			)
-			(layer "Eco1.User")
-		)
-		(fp_line
-			(start -15.313 6.77)
-			(end -8.563 6.77)
-			(stroke
-				(width 0.1)
-				(type solid)
-			)
-			(layer "Eco1.User")
-		)
-		(fp_line
-			(start -8.563 -5.53)
-			(end -15.313 -5.53)
-			(stroke
-				(width 0.1)
-				(type solid)
-			)
-			(layer "Eco1.User")
-		)
-		(fp_line
-			(start -8.563 6.77)
-			(end -8.563 -5.53)
-			(stroke
-				(width 0.1)
-				(type solid)
-			)
-			(layer "Eco1.User")
-		)
-		(fp_line
-			(start 8.563 -5.53)
-			(end 8.563 6.77)
-			(stroke
-				(width 0.1)
-				(type solid)
-			)
-			(layer "Eco1.User")
-		)
-		(fp_line
-			(start 8.563 6.77)
-			(end 15.313 6.77)
-			(stroke
-				(width 0.1)
-				(type solid)
-			)
-			(layer "Eco1.User")
-		)
-		(fp_line
-			(start 15.313 -5.53)
-			(end 8.563 -5.53)
-			(stroke
-				(width 0.1)
-				(type solid)
-			)
-			(layer "Eco1.User")
-		)
-		(fp_line
-			(start 15.313 6.77)
-			(end 15.313 -5.53)
-			(stroke
-				(width 0.1)
-				(type solid)
-			)
-			(layer "Eco1.User")
-		)
-		(fp_text user "${REFERENCE}"
-			(at 0 0 0)
-			(layer "F.Fab")
-			(effects
-				(font
-					(size 1 1)
-					(thickness 0.15)
-				)
-			)
-		)
-		(pad "" np_thru_hole circle
-			(at -11.938 -6.985)
-			(size 3.048 3.048)
-			(drill 3.048)
-			(layers "*.Cu" "*.Mask")
-		)
-		(pad "" np_thru_hole circle
-			(at -11.938 8.225)
-			(size 3.9878 3.9878)
-			(drill 3.9878)
-			(layers "*.Cu" "*.Mask")
-		)
-		(pad "" np_thru_hole circle
-			(at 11.938 -6.985)
-			(size 3.048 3.048)
-			(drill 3.048)
-			(layers "*.Cu" "*.Mask")
-		)
-		(pad "" np_thru_hole circle
-			(at 11.938 8.225)
-			(size 3.9878 3.9878)
-			(drill 3.9878)
-			(layers "*.Cu" "*.Mask")
-		)
-		(embedded_fonts no)
-		(model "${SCOTTOKEEBS_KICAD}/3dmodels/ScottoKeebs_Stabilizer.3dshapes/Stabilizer_MX_2.00u.step"
-			(offset
-				(xyz 0 0 0)
-			)
-			(scale
-				(xyz 1 1 1)
-			)
-			(rotate
-				(xyz 0 0 0)
-			)
-		)
-	)
 	(footprint "ScottoKeebs_MX:MX_PCB_1.00u"
 		(layer "F.Cu")
@@
 	)
 	(segment
-		(start 248.6398 -54.9648)
-		(end 243.84 -50.165)
-		(width 0.2)
-		(layer "B.Cu")
-		(net "COL12")
-	)
-	(segment
 		(start 225.3681 -125.4185)
 		(end 225.3681 -132.4668)
@@
 	)
 	(segment
-		(start 251.1492 -88.0996)
-		(end 251.1492 -75.7668)
-		(width 0.2)
-		(layer "B.Cu")
-		(net "COL12")
-	)
-	(segment
-		(start 251.1492 -75.7668)
-		(end 248.6398 -73.2574)
-		(width 0.2)
-		(layer "B.Cu")
-		(net "COL12")
-	)
-	(segment
 		(start -13.34375 -114.75625)
 		(end -15.7375 -112.3625)
@@
 	)
 	(segment
-		(start 248.6398 -73.2574)
-		(end 248.6398 -54.9648)
+		(start 238.3673 -88.265)
+		(end 236.6963 -89.936)
 		(width 0.2)
 		(layer "B.Cu")
@@
 	)
 	(segment
+		(start 250.9838 -88.265)
+		(end 238.3673 -88.265)
+		(width 0.2)
+		(layer "B.Cu")
+		(net "COL12")
+	)
+	(segment
 		(start 225.3681 -115.0393)
 		(end 225.3681 -113.5359)
@@
 	(segment
 		(start 255.3782 -88.8281)
-		(end 257.3565 -86.8498)
+		(end 257.232838 -86.973463)
 		(width 0.2)
 		(layer "B.Cu")
@@
 	)
 	(segment
-		(start 257.3565 -55.6985)
-		(end 262.89 -50.165)
+		(start 251.46 -138.43)
+		(end 258.445 -145.415)
 		(width 0.2)
 		(layer "B.Cu")
@@
 	)
 	(segment
-		(start 251.46 -138.43)
-		(end 258.445 -145.415)
+		(start 258.1275 -107.315)
+		(end 255.3782 -107.315)
 		(width 0.2)
 		(layer "B.Cu")
@@
 	)
 	(segment
-		(start 257.3565 -86.8498)
-		(end 257.3565 -55.6985)
+		(start 258.445 -145.415)
+		(end 262.89 -145.415)
 		(width 0.2)
 		(layer "B.Cu")
@@
 	)
 	(segment
-		(start 258.1275 -107.315)
-		(end 255.3782 -107.315)
+		(start 257.232838 -74.872162)
+		(end 262.89 -69.215)
 		(width 0.2)
 		(layer "B.Cu")
@@
 	)
 	(segment
-		(start 258.445 -145.415)
-		(end 262.89 -145.415)
+		(start 48.888766 -111.514625)
+		(end 50.005441 -112.6313)
 		(width 0.2)
 		(layer "B.Cu")
@@
 	)
 	(segment
-		(start 48.888766 -111.514625)
-		(end 50.005441 -112.6313)
+		(start 262.89 -69.215)
+		(end 262.89 -50.165)
+		(width 0.2)
+		(layer "B.Cu")
+		(net "COL13")
+	)
+	(segment
+		(start 257.232838 -86.973463)
+		(end 257.3565 -86.8498)
 		(width 0.2)
 		(layer "B.Cu")
@@
 		(width 0.2)
 		(layer "B.Cu")
+		(net "COL13")
+	)
+	(segment
+		(start 257.232838 -86.973463)
+		(end 257.232838 -74.872162)
+		(width 0.2)
+		(layer "B.Cu")
