File: PCB/PepuinoNova75.kicad_sch (KiCad schematic)
At the start: 172 parts, among them SW1 Switch, SW10 Switch, SW11 Switch, SW12 Switch, SW13 Switch, SW14 Switch, SW15 Switch, SW16 Switch, SW17 Switch, SW18 Switch, SW19 Switch, SW2 Switch, SW20 Switch, SW21 Switch, SW22 Switch, SW23 Switch, SW24 Switch, SW25 Switch, SW26 Switch, SW27 Switch, SW28 Switch, SW29 Switch, SW3 Switch, SW30 Switch, SW31 Switch, SW32 Switch, SW33 Switch, SW34 Switch, SW35 Switch, SW36 Switch, SW37 Switch, SW38 Switch, SW39 Switch, SW4 Switch, SW40 Switch, SW41 Switch, SW42 Switch, SW43 Switch, SW44 Switch, SW45 Switch, SW46 Switch, SW47 Switch, SW48 Switch, SW49 Switch, SW5 Switch, SW50 Switch, SW51 Switch, SW52 Switch, SW53 Switch, SW54 Switch, SW55 Switch, SW56 Switch, SW57 Switch, SW58 Switch, SW59 Switch, SW6 Switch, SW60 Switch, SW61 Switch, SW62 Switch, SW63 Switch, SW64 Switch, SW65 Switch, SW66 Switch, SW67 Switch, SW68 Switch, SW69 Switch, SW7 Switch, SW71 Switch, SW72 Switch, SW73 Switch, SW74 Switch, SW75 Switch, SW76 Switch, SW77 Switch, SW78 Switch, SW79 Switch, SW8 Switch, SW80 Switch, SW81 Switch, SW82 Switch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

Commit message: fix fatal error in pcb +  fix case + update images
Parts:
- removed S5: MX_stab, ScottoKeebs_Stabilizers:Stabilizer_MX_2.00u, symbol PCM_marbastlib-mx:MX_stab
Connections:
- net COL13: now also SW72.1
Other:
- moved on the sheet: D72, SW72
Changed lines of the file:
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@@
 	)
 	(junction
+		(at 242.57 148.59)
+		(diameter 0)
+		(color 0 0 0 0)
+	)
+	(junction
 		(at 34.29 128.27)
 		(diameter 0)
@@
 	)
 	(junction
+		(at 232.41 143.51)
+		(diameter 0)
+		(color 0 0 0 0)
+	)
+	(junction
 		(at 247.65 143.51)
 		(diameter 0)
@@
 	)
 	(junction
-		(at 243.84 148.59)
-		(diameter 0)
-		(color 0 0 0 0)
-	)
-	(junction
 		(at 186.69 128.27)
 		(diameter 0)
@@
 	(wire
 		(pts
+			(xy 232.41 143.51) (xy 232.41 160.02)
+		)
+		(stroke
+			(width 0)
+			(type default)
+		)
+	)
+	(wire
+		(pts
 			(xy 247.65 82.55) (xy 252.73 82.55)
 		)
@@
 	(wire
 		(pts
-			(xy 232.41 113.03) (xy 232.41 160.02)
+			(xy 232.41 113.03) (xy 232.41 143.51)
 		)
 		(stroke
@@
 	(wire
 		(pts
+			(xy 242.57 148.59) (xy 257.81 148.59)
+		)
+		(stroke
+			(width 0)
+			(type default)
+		)
+	)
+	(wire
+		(pts
 			(xy 247.65 97.79) (xy 247.65 113.03)
 		)
@@
 	(wire
 		(pts
-			(xy 227.33 148.59) (xy 243.84 148.59)
+			(xy 227.33 148.59) (xy 242.57 148.59)
 		)
 		(stroke
@@
 	(wire
 		(pts
-			(xy 243.84 148.59) (xy 257.81 148.59)
-		)
-		(stroke
-			(width 0)
-			(type default)
-		)
-	)
-	(wire
-		(pts
 			(xy 24.13 165.1) (xy 44.45 165.1)
 		)
@@
 	)
 	(symbol
-		(lib_id "PCM_marbastlib-mx:MX_stab")
-		(at 62.23 46.99 0)
-		(unit 1)
-		(body_style 1)
-		(exclude_from_sim no)
-		(in_bom yes)
-		(on_board yes)
-		(in_pos_files yes)
-		(dnp no)
-		(fields_autoplaced yes)
-		(property "Reference" "S5"
-			(at 68.58 45.5929 0)
-			(show_name no)
-			(do_not_autoplace no)
-			(effects
-				(font
-					(size 1.27 1.27)
-				)
-				(justify left)
-			)
-		)
-		(property "Value" "MX_stab"
-			(at 68.58 48.1329 0)
-			(show_name no)
-			(do_not_autoplace no)
-			(effects
-				(font
-					(size 1.27 1.27)
-				)
-				(justify left)
-			)
-		)
-		(property "Footprint" "ScottoKeebs_Stabilizers:Stabilizer_MX_2.00u"
-			(at 62.23 46.99 0)
-			(hide yes)
-			(show_name no)
-			(do_not_autoplace no)
-			(effects
-				(font
-					(size 1.27 1.27)
-				)
-			)
-		)
-		(property "Datasheet" ""
-			(at 62.23 46.99 0)
-			(hide yes)
-			(show_name no)
-			(do_not_autoplace no)
-			(effects
-				(font
-					(size 1.27 1.27)
-				)
-			)
-		)
-		(property "Description" "Cherry MX-style stabilizer"
-			(at 62.23 46.99 0)
-			(hide yes)
-			(show_name no)
-			(do_not_autoplace no)
-			(effects
-				(font
-					(size 1.27 1.27)
-				)
-			)
-		)
-		(instances
-			(project "PepuinoNova75"
-				(path "/ce63fa7b-8e8c-4088-a358-a5b5a66994c2"
-					(reference "S5")
-					(unit 1)
-				)
-			)
-		)
-	)
-	(symbol
 		(lib_id "ScottoKeebs:Placeholder_Diode")
 		(at 242.57 100.33 0)
@@
 	(symbol
 		(lib_id "ScottoKeebs:Placeholder_Diode")
-		(at 243.84 146.05 0)
+		(at 242.57 146.05 0)
 		(unit 1)
 		(body_style 1)
@@
 		(fields_autoplaced yes)
 		(property "Reference" "D72"
-			(at 243.69 144.984 0)
+			(at 242.42 144.984 0)
 			(show_name no)
 			(do_not_autoplace yes)
@@
 		)
 		(property "Value" ""
-			(at 246.38 146.0499 0)
+			(at 245.11 146.0499 0)
 			(show_name no)
 			(do_not_autoplace no)
@@
 		)
 		(property "Footprint" "ScottoKeebs_Components:Diode_SOD-123"
-			(at 243.84 146.05 90)
+			(at 242.57 146.05 90)
 			(hide yes)
 			(show_name no)
@@
 		)
 		(property "Datasheet" ""
-			(at 243.84 146.05 90)
+			(at 242.57 146.05 90)
 			(hide yes)
 			(show_name no)
@@
 		)
 		(property "Description" ""
-			(at 247.65 146.05 90)
+			(at 246.38 146.05 90)
 			(hide yes)
 			(show_name no)
@@
 	(symbol
 		(lib_id "ScottoKeebs:Placeholder_Switch")
-		(at 238.76 143.51 0)
+		(at 237.49 143.51 0)
 		(unit 1)
 		(body_style 1)
@@
 		(fields_autoplaced yes)
 		(property "Reference" "SW72"
-			(at 238.76 135.89 0)
+			(at 237.49 135.89 0)
 			(show_name no)
 			(do_not_autoplace no)
@@
 		)
 		(property "Value" "Switch"
-			(at 238.76 138.43 0)
+			(at 237.49 138.43 0)
 			(show_name no)
 			(do_not_autoplace no)
@@
 		)
 		(property "Footprint" "ScottoKeebs_MX:MX_PCB_1.00u"
-			(at 238.76 138.43 0)
+			(at 237.49 138.43 0)
 			(hide yes)
 			(show_name no)
@@
 		)
 		(property "Datasheet" ""
-			(at 238.76 138.43 0)
+			(at 237.49 138.43 0)
 			(hide yes)
 			(show_name no)
@@
 		)
 		(property "Description" "Push button switch, generic, two pins"
-			(at 238.76 143.51 0)
+			(at 237.49 143.51 0)
 			(hide yes)
 			(show_name no)
